File: PCB/Keyboard/Keyboard.kicad_pcb (KiCad board)
At the start: 2 copper layers, 285.8 x 95.2 mm, 146 parts, among them J1 USB_C_Receptacle_USB2.0, U1 STM32F072CBT6, U2 PRTR5V0U2X, U3 XC6206PxxxMR-Regulator_Linear

Commit message: wire rows and cols
Parts:
- moved S3 185.3 mm to (136.8, 170.0), turned to 0 degrees
- moved S2 85.5 mm to (82.9, 168.5), turned to 0 degrees
- moved S1 60.6 mm to (111.5, 142.0), turned to 0 degrees
- moved C1 28.9 mm to (201.3, 168.2)
- moved C7 28.9 mm to (201.3, 167.0)
- moved BOOT1 28.9 mm to (205.8, 177.5)
- moved C10 28.9 mm to (205.6, 152.8)
- moved C2 28.9 mm to (208.3, 153.0)
- moved C3 28.9 mm to (207.1, 156.0)
- moved C4 28.9 mm to (198.3, 156.3)
- moved C5 28.9 mm to (207.3, 164.8)
- moved C6 28.9 mm to (206.8, 166.3)
- moved C8 28.9 mm to (205.8, 146.0)
- moved C9 28.9 mm to (204.3, 149.3)
- moved F1 28.9 mm to (202.8, 147.0)
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Connections:
- D1 pad 1: unconnected-(D1-K-Pad1) -> ROW0
- D10 pad 1: unconnected-(D10-K-Pad1) -> ROW0
- D11 pad 1: unconnected-(D11-K-Pad1) -> ROW0
- D12 pad 1: unconnected-(D12-K-Pad1) -> ROW0
- D13 pad 1: unconnected-(D13-K-Pad1) -> ROW0
- D14 pad 1: unconnected-(D14-K-Pad1) -> ROW0
- D15 pad 1: unconnected-(D15-K-Pad1) -> ROW0
- D16 pad 1: unconnected-(D16-K-Pad1) -> ROW1
- D17 pad 1: unconnected-(D17-K-Pad1) -> ROW1
- D18 pad 1: unconnected-(D18-K-Pad1) -> ROW1
- D19 pad 1: unconnected-(D19-K-Pad1) -> ROW1
- D2 pad 1: unconnected-(D2-K-Pad1) -> ROW0
- D20 pad 1: unconnected-(D20-K-Pad1) -> ROW1
- D21 pad 1: unconnected-(D21-K-Pad1) -> ROW1
- D22 pad 1: unconnected-(D22-K-Pad1) -> ROW1
- D23 pad 1: unconnected-(D23-K-Pad1) -> ROW1
- D24 pad 1: unconnected-(D24-K-Pad1) -> ROW1
- D25 pad 1: unconnected-(D25-K-Pad1) -> ROW1
- D26 pad 1: unconnected-(D26-K-Pad1) -> ROW1
- D27 pad 1: unconnected-(D27-K-Pad1) -> ROW1
- D28 pad 1: unconnected-(D28-K-Pad1) -> ROW1
- D29 pad 1: unconnected-(D29-K-Pad1) -> ROW1
- D3 pad 1: unconnected-(D3-K-Pad1) -> ROW0
- D30 pad 1: unconnected-(D30-K-Pad1) -> ROW2
- D31 pad 1: unconnected-(D31-K-Pad1) -> ROW2
- D32 pad 1: unconnected-(D32-K-Pad1) -> ROW2
- D33 pad 1: unconnected-(D33-K-Pad1) -> ROW2
- D34 pad 1: unconnected-(D34-K-Pad1) -> ROW2
- D35 pad 1: unconnected-(D35-K-Pad1) -> ROW2
- D36 pad 1: unconnected-(D36-K-Pad1) -> ROW2
- D37 pad 1: unconnected-(D37-K-Pad1) -> ROW2
- D38 pad 1: unconnected-(D38-K-Pad1) -> ROW2
- D39 pad 1: unconnected-(D39-K-Pad1) -> ROW2
- D4 pad 1: unconnected-(D4-K-Pad1) -> ROW0
- D40 pad 1: unconnected-(D40-K-Pad1) -> ROW2
- D41 pad 1: unconnected-(D41-K-Pad1) -> ROW2
- D42 pad 1: unconnected-(D42-K-Pad1) -> ROW2
- D43 pad 1: unconnected-(D43-K-Pad1) -> ROW3
- D44 pad 1: unconnected-(D44-K-Pad1) -> ROW3
- D45 pad 1: unconnected-(D45-K-Pad1) -> ROW3
- D46 pad 1: unconnected-(D46-K-Pad1) -> ROW3
- D47 pad 1: unconnected-(D47-K-Pad1) -> ROW3
- D48 pad 1: unconnected-(D48-K-Pad1) -> ROW3
- D49 pad 1: unconnected-(D49-K-Pad1) -> ROW3
- D5 pad 1: unconnected-(D5-K-Pad1) -> ROW0
- D50 pad 1: unconnected-(D50-K-Pad1) -> ROW3
- D51 pad 1: unconnected-(D51-K-Pad1) -> ROW3
- D52 pad 1: unconnected-(D52-K-Pad1) -> ROW3
- D53 pad 1: unconnected-(D53-K-Pad1) -> ROW3
- D54 pad 1: unconnected-(D54-K-Pad1) -> ROW3
- D55 pad 1: unconnected-(D55-K-Pad1) -> ROW3
- D56 pad 1: unconnected-(D56-K-Pad1) -> ROW4
- D57 pad 1: unconnected-(D57-K-Pad1) -> ROW4
- D58 pad 1: unconnected-(D58-K-Pad1) -> ROW4
- D59 pad 1: unconnected-(D59-K-Pad1) -> ROW4
- D6 pad 1: unconnected-(D6-K-Pad1) -> ROW0
- D60 pad 1: unconnected-(D60-K-Pad1) -> ROW4
- D61 pad 1: unconnected-(D61-K-Pad1) -> ROW4
- D7 pad 1: unconnected-(D7-K-Pad1) -> ROW0
- D8 pad 1: unconnected-(D8-K-Pad1) -> ROW0
- D9 pad 1: unconnected-(D9-K-Pad1) -> ROW0
- MX1 pad 1: unconnected-(MX1-Pad1) -> COL0
- MX10 pad 1: unconnected-(MX10-Pad1) -> COL9
- MX11 pad 1: unconnected-(MX11-Pad1) -> COL10
- MX12 pad 1: unconnected-(MX12-Pad1) -> COL11
- MX13 pad 1: unconnected-(MX13-Pad1) -> COL12
- MX14 pad 1: unconnected-(MX14-Pad1) -> COL13
- MX15 pad 1: unconnected-(MX15-Pad1) -> COL14
- MX16 pad 1: unconnected-(MX16-Pad1) -> COL0
- MX17 pad 1: unconnected-(MX17-Pad1) -> COL1
- MX18 pad 1: unconnected-(MX18-Pad1) -> COL2
- MX19 pad 1: unconnected-(MX19-Pad1) -> COL3
- MX2 pad 1: unconnected-(MX2-Pad1) -> COL1
- MX20 pad 1: unconnected-(MX20-Pad1) -> COL4
- MX21 pad 1: unconnected-(MX21-Pad1) -> COL5
- MX22 pad 1: unconnected-(MX22-Pad1) -> COL6
- MX23 pad 1: unconnected-(MX23-Pad1) -> COL7
- MX24 pad 1: unconnected-(MX24-Pad1) -> COL8
- MX25 pad 1: unconnected-(MX25-Pad1) -> COL9
- MX26 pad 1: unconnected-(MX26-Pad1) -> COL10
- MX27 pad 1: unconnected-(MX27-Pad1) -> COL11
- MX28 pad 1: unconnected-(MX28-Pad1) -> COL12
- MX29 pad 1: unconnected-(MX29-Pad1) -> COL13
- MX3 pad 1: unconnected-(MX3-Pad1) -> COL2
- MX30 pad 1: unconnected-(MX30-Pad1) -> COL0
- MX31 pad 1: unconnected-(MX31-Pad1) -> COL1
- MX32 pad 1: unconnected-(MX32-Pad1) -> COL2
- MX33 pad 1: unconnected-(MX33-Pad1) -> COL3
- MX34 pad 1: unconnected-(MX34-Pad1) -> COL4
- MX35 pad 1: unconnected-(MX35-Pad1) -> COL5
- MX36 pad 1: unconnected-(MX36-Pad1) -> COL6
- MX37 pad 1: unconnected-(MX37-Pad1) -> COL7
- MX38 pad 1: unconnected-(MX38-Pad1) -> COL8
- MX39 pad 1: unconnected-(MX39-Pad1) -> COL9
- MX4 pad 1: unconnected-(MX4-Pad1) -> COL3
- MX40 pad 1: unconnected-(MX40-Pad1) -> COL10
- MX41 pad 1: unconnected-(MX41-Pad1) -> COL11
- MX42 pad 1: unconnected-(MX42-Pad1) -> COL12
- MX43 pad 1: unconnected-(MX43-Pad1) -> COL0
- MX44 pad 1: unconnected-(MX44-Pad1) -> COL1
- MX45 pad 1: unconnected-(MX45-Pad1) -> COL2
- MX46 pad 1: unconnected-(MX46-Pad1) -> COL3
- MX47 pad 1: unconnected-(MX47-Pad1) -> COL4
- MX48 pad 1: unconnected-(MX48-Pad1) -> COL5
- MX49 pad 1: unconnected-(MX49-Pad1) -> COL6
- MX5 pad 1: unconnected-(MX5-Pad1) -> COL4
- MX50 pad 1: unconnected-(MX50-Pad1) -> COL7
- MX51 pad 1: unconnected-(MX51-Pad1) -> COL8
- MX52 pad 1: unconnected-(MX52-Pad1) -> COL9
- MX53 pad 1: unconnected-(MX53-Pad1) -> COL10
- MX54 pad 1: unconnected-(MX54-Pad1) -> COL11
- MX55 pad 1: unconnected-(MX55-Pad1) -> COL14
- MX56 pad 1: unconnected-(MX56-Pad1) -> COL0
- MX57 pad 1: unconnected-(MX57-Pad1) -> COL1
- MX58 pad 1: unconnected-(MX58-Pad1) -> COL2
- MX59 pad 1: unconnected-(MX59-Pad1) -> COL5
- MX6 pad 1: unconnected-(MX6-Pad1) -> COL5
- MX60 pad 1: unconnected-(MX60-Pad1) -> COL9
- MX61 pad 1: unconnected-(MX61-Pad1) -> COL10
- MX7 pad 1: unconnected-(MX7-Pad1) -> COL6
- MX8 pad 1: unconnected-(MX8-Pad1) -> COL7
- MX9 pad 1: unconnected-(MX9-Pad1) -> COL8
Routing:
- net ROW0: track 0.00 -> 266.7 mm
- net ROW1: track 0.00 -> 257.2 mm
- net ROW3: track 0.00 -> 254.8 mm
- net ROW2: track 0.00 -> 247.7 mm
- net ROW4: track 0.00 -> 214.3 mm
- net COL1: track 0.00 -> 92.9 mm
- net COL2: track 0.00 -> 90.0 mm
- net COL5: track 0.00 -> 88.0 mm
- net COL10: track 0.00 -> 88.0 mm
- net COL9: track 0.00 -> 86.1 mm
- net COL0: track 0.00 -> 84.1 mm
- net COL11: track 0.00 -> 70.0 mm
- net COL7: track 0.00 -> 68.7 mm
- net COL8: track 0.00 -> 67.0 mm
- net COL6: track 0.00 -> 67.0 mm
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Other:
- outline, holes or cut-outs redrawn
