File: PCB/Keyboard/Keyboard.kicad_pcb (KiCad board)
At the start: 2 copper layers, 285.8 x 95.2 mm, 146 parts, among them J1 USB_C_Receptacle_USB2.0, U1 STM32F072CBT6, U2 PRTR5V0U2X, U3 XC6206PxxxMR-Regulator_Linear

Commit message: Finalize slider PCB
Parts:
- moved S2 231.9 mm to (293.1, 70.5), turned to 180 degrees
- moved S3 118.3 mm to (50.2, 89.5), turned to 180 degrees
- moved S1 60.6 mm to (162.1, 108.6), turned to 180 degrees

Commit message: organize stm32
Parts:
- moved C8 148.6 mm to (186.0, -1.30)
- moved C9 148.6 mm to (184.5, 1.95)
- moved F1 148.6 mm to (183.0, -0.30)
- moved J1 148.6 mm to (183.0, -12.6)
- moved R1 148.6 mm to (186.0, -3.30)
- moved R2 148.6 mm to (186.0, -5.80)
- moved U2 148.6 mm to (183.0, -4.55)
- moved C2 148.5 mm to (187.2, 6.04)
- moved C10 148.3 mm to (184.4, 6.00)
- moved U3 148.3 mm to (185.9, 3.50)
- moved D59 10.2 mm to (170.1, 99.6), turned to -90 degrees
- moved D8 4.98 mm to (174.8, 35.5)
Routing:
- net NRST: track 56.2 -> 19.5 mm
- net BOOT0: track 47.3 -> 25.6 mm
- net /A10: track 26.3 -> 5.24 mm
- net /A9: track 23.5 -> 5.13 mm
- net /A8: track 20.8 -> 5.11 mm
- net ROW0: track 266.7 -> 280.4 mm
- net ROW4: track 214.3 -> 227.7 mm
- net /B15: track 18.0 -> 5.09 mm
- net +3V3: track 78.1 -> 65.3 mm, vias 6 -> 4
- net /A0: track 20.5 -> 7.78 mm
- net VBUS: track 27.7 -> 16.0 mm
- net /A1: track 17.8 -> 7.08 mm
- net /A13: track 16.0 -> 5.61 mm
- net /B14: track 15.3 -> 4.94 mm
- net /A3: track 13.2 -> 3.53 mm
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
Commit message: wire stm32
Parts:
- moved RST1 94.4 mm to (138.9, 105.5), turned to 0 degrees
- moved BOOT1 94.1 mm to (138.9, 111.5), turned to 180 degrees
- moved C1 55.9 mm to (189.9, 113.5)
- moved C7 55.9 mm to (189.9, 112.3)
- moved C3 55.9 mm to (195.7, 101.3)
- moved C4 55.9 mm to (186.9, 101.5)
- moved C5 55.9 mm to (195.9, 110.0)
- moved C6 55.9 mm to (195.4, 111.5)
- moved R3 55.9 mm to (192.7, 115.8)
- moved R4 55.9 mm to (190.2, 115.8)
- moved U1 55.9 mm to (191.4, 105.8)
- moved C10 17.1 mm to (184.3, -11.1)
- moved C2 15.9 mm to (185.8, -9.80)
- moved U3 15.8 mm to (186.3, -12.3)
- moved C9 15.6 mm to (184.3, -13.6), turned to 0 degrees
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Routing:
- net BOOT0: track 25.6 -> 74.8 mm
- net NRST: track 19.5 -> 65.2 mm
- net +3V3: track 65.3 -> 103.7 mm
- net GND: track 155.2 -> 187.6 mm, vias 8 -> 7
- net /A13: track 5.61 -> 3.33 mm
- net /A10: track 5.24 -> 3.50 mm
- net /B13: track 5.08 -> 3.40 mm
- net /A8: track 5.11 -> 3.46 mm
- net /A9: track 5.13 -> 3.48 mm
- net /B12: track 5.03 -> 3.37 mm
- net /B15: track 5.09 -> 3.44 mm
- net D-: track 21.0 -> 19.5 mm
- net /B14: track 4.94 -> 3.44 mm
- net D+: track 22.6 -> 21.8 mm
- net +5V: track 10.4 -> 9.64 mm
