File: PCB/TMR slider module/slider.kicad_sch (KiCad schematic)
At the start: 6 parts, among them J1 Conn_01x03_Socket, U1 CT8510

Commit message: Finalize slider PCB
Parts:
- added H1, H2, H3, H4: MountingHole, MountingHole:MountingHole_2.2mm_M2, symbol Mechanical:MountingHole
- U1: value CT8510 -> A1324; footprint Package_TO_SOT_SMD:SOT-23-3 -> Package_TO_SOT_SMD:SOT-23W
